File: FelinaePurr.sch (KiCad schematic (older format))
At the start: 24 parts, among them P1 USB_OTG, P2 JACK, U1 FT232RL, U2 SN74LVC1G125-Q1

Commit message: USB-A Version
Parts:
- removed P1: USB_OTG, Connect:USB_Micro-B, symbol USB_OTG
- added P1: USB_A, PadsLib:MC32603_USB_A, symbol USB_A
Connections:
- net +5VD: now also P1.1 (VCC)
- net GND: now also P1.4 (GND), P1.5 (shield)
- net Dm renamed D-
- net D-: now also P1.2 (D-)
- net Dp renamed D+
- net D+: now also P1.3 (D+)
- no-connect marks 15 -> 14
Changed lines of the file:
@@
 $EndDescr
-$Comp
-L USB_OTG P1
-U 1 1 5788BE50
-P 3600 4000
-F 0 "P1" H 3676 4325 50  0000 C CNN
-F 1 "USB_OTG" H 3676 4234 50  0000 C CNN
-F 2 "Connect:USB_Micro-B" V 3550 3900 50  0001 C CNN
-F 3 "" V 3550 3900 50  0000 C CNN
-	1    3600 4000
-	1    0    0    -1
-$EndComp
 $Comp
 L CONN_01X03 P2
@@
 $EndComp
 $Comp
-L +5V #PWR4
+L +5V #PWR01
 U 1 1 5788C03E
 P 2500 1550
-F 0 "#PWR4" H 2500 1400 50  0001 C CNN
+F 0 "#PWR01" H 2500 1400 50  0001 C CNN
 F 1 "+5V" H 2515 1723 50  0000 C CNN
 F 2 "" H 2500 1550 50  0000 C CNN
@@
 $EndComp
 $Comp
-L +5VD #PWR2
+L +5VD #PWR02
 U 1 1 5788C095
 P 2150 1750
-F 0 "#PWR2" H 2150 1600 50  0001 C CNN
+F 0 "#PWR02" H 2150 1600 50  0001 C CNN
 F 1 "+5VD" H 2165 1923 50  0000 C CNN
 F 2 "" H 2150 1750 50  0000 C CNN
@@
 $EndComp
 $Comp
-L +5VL #PWR7
+L +5VL #PWR03
 U 1 1 5788C0B2
 P 2850 1750
-F 0 "#PWR7" H 2850 1600 50  0001 C CNN
+F 0 "#PWR03" H 2850 1600 50  0001 C CNN
 F 1 "+5VL" H 2865 1923 50  0000 C CNN
 F 2 "" H 2850 1750 50  0000 C CNN
@@
 $EndComp
 $Comp
-L PWR_FLAG #FLG1
+L PWR_FLAG #FLG04
 U 1 1 5788C17B
 P 2450 1750
-F 0 "#FLG1" H 2450 1845 50  0001 C CNN
+F 0 "#FLG04" H 2450 1845 50  0001 C CNN
 F 1 "PWR_FLAG" V 2750 1800 50  0000 L CNN
 F 2 "" H 2450 1750 50  0000 C CNN
@@
 $EndComp
 $Comp
-L +5VL #PWR19
+L +5VL #PWR05
 U 1 1 5788C270
 P 9050 4650
-F 0 "#PWR19" H 9050 4500 50  0001 C CNN
+F 0 "#PWR05" H 9050 4500 50  0001 C CNN
 F 1 "+5VL" H 9065 4823 50  0000 C CNN
 F 2 "" H 9050 4650 50  0000 C CNN
@@
 $EndComp
 $Comp
-L GND #PWR20
+L GND #PWR06
 U 1 1 5788C2A8
 P 9050 5050
-F 0 "#PWR20" H 9050 4800 50  0001 C CNN
+F 0 "#PWR06" H 9050 4800 50  0001 C CNN
 F 1 "GND" H 9055 4877 50  0000 C CNN
 F 2 "" H 9050 5050 50  0000 C CNN
@@
 TIP\nINNER\nBASE
 $Comp
-L PWR_FLAG #FLG2
+L PWR_FLAG #FLG07
 U 1 1 5788C38F
 P 8850 4750
-F 0 "#FLG2" H 8850 4845 50  0001 C CNN
+F 0 "#FLG07" H 8850 4845 50  0001 C CNN
 F 1 "PWR_FLAG" V 8850 4928 50  0000 L CNN
 F 2 "" H 8850 4750 50  0000 C CNN
@@
 $EndComp
 $Comp
-L GND #PWR16
+L GND #PWR08
 U 1 1 5788C66D
 P 7250 2300
-F 0 "#PWR16" H 7250 2050 50  0001 C CNN
+F 0 "#PWR08" H 7250 2050 50  0001 C CNN
 F 1 "GND" H 7255 2127 50  0000 C CNN
 F 2 "" H 7250 2300 50  0000 C CNN
@@
 $EndComp
 $Comp
-L +5VD #PWR5
+L +5VD #PWR09
 U 1 1 5788CC48
 P 2500 4250
-F 0 "#PWR5" H 2500 4100 50  0001 C CNN
+F 0 "#PWR09" H 2500 4100 50  0001 C CNN
 F 1 "+5VD" H 2515 4423 50  0000 C CNN
 F 2 "" H 2500 4250 50  0000 C CNN
@@
 $EndComp
 $Comp
-L GND #PWR9
+L GND #PWR010
 U 1 1 5788CC92
-P 3800 4450
-F 0 "#PWR9" H 3800 4200 50  0001 C CNN
-F 1 "GND" H 3805 4277 50  0000 C CNN
-F 2 "" H 3800 4450 50  0000 C CNN
-F 3 "" H 3800 4450 50  0000 C CNN
-	1    3800 4450
-	1    0    0    -1
-$EndComp
-NoConn ~ 3700 4300
+P 3700 4450
+F 0 "#PWR010" H 3700 4200 50  0001 C CNN
+F 1 "GND" H 3705 4277 50  0000 C CNN
+F 2 "" H 3700 4450 50  0000 C CNN
+F 3 "" H 3700 4450 50  0000 C CNN
+	1    3700 4450
+	1    0    0    -1
+$EndComp
 $Comp
 L C C1
@@
 $EndComp
 $Comp
-L GND #PWR3
+L GND #PWR011
 U 1 1 5788D07A
 P 2450 6100
-F 0 "#PWR3" H 2450 5850 50  0001 C CNN
+F 0 "#PWR011" H 2450 5850 50  0001 C CNN
 F 1 "GND" H 2455 5927 50  0000 C CNN
 F 2 "" H 2450 6100 50  0000 C CNN
@@
 $EndComp
 $Comp
-L GND #PWR1
+L GND #PWR012
 U 1 1 5788D0D6
 P 1600 5800
-F 0 "#PWR1" H 1600 5550 50  0001 C CNN
+F 0 "#PWR012" H 1600 5550 50  0001 C CNN
 F 1 "GND" H 1605 5627 50  0000 C CNN
 F 2 "" H 1600 5800 50  0000 C CNN
@@
 $EndComp
 $Comp
-L +5VD #PWR10
+L +5VD #PWR013
 U 1 1 5788D588
 P 4450 3650
-F 0 "#PWR10" H 4450 3500 50  0001 C CNN
+F 0 "#PWR013" H 4450 3500 50  0001 C CNN
 F 1 "+5VD" H 4465 3823 50  0000 C CNN
 F 2 "" H 4450 3650 50  0000 C CNN
@@
 $EndComp
 $Comp
-L GND #PWR12
+L GND #PWR014
 U 1 1 5788DEA1
 P 5050 5200
-F 0 "#PWR12" H 5050 4950 50  0001 C CNN
+F 0 "#PWR014" H 5050 4950 50  0001 C CNN
 F 1 "GND" H 5055 5027 50  0000 C CNN
 F 2 "" H 5050 5200 50  0000 C CNN
@@
 $EndComp
 $Comp
-L +5VD #PWR11
+L +5VD #PWR015
 U 1 1 5788E141
 P 4900 3650
-F 0 "#PWR11" H 4900 3500 50  0001 C CNN
+F 0 "#PWR015" H 4900 3500 50  0001 C CNN
 F 1 "+5VD" H 4915 3823 50  0000 C CNN
 F 2 "" H 4900 3650 50  0000 C CNN
@@
 $EndComp
 $Comp
-L +5VL #PWR13
+L +5VL #PWR016
 U 1 1 5788E182
 P 5200 3650
-F 0 "#PWR13" H 5200 3500 50  0001 C CNN
+F 0 "#PWR016" H 5200 3500 50  0001 C CNN
 F 1 "+5VL" H 5215 3823 50  0000 C CNN
 F 2 "" H 5200 3650 50  0000 C CNN
@@
 $EndComp
 $Comp
-L GND #PWR8
+L GND #PWR017
 U 1 1 5788ECC9
 P 2850 4900
-F 0 "#PWR8" H 2850 4650 50  0001 C CNN
+F 0 "#PWR017" H 2850 4650 50  0001 C CNN
 F 1 "GND" H 2855 4727 50  0000 C CNN
 F 2 "" H 2850 4900 50  0000 C CNN
@@
 $EndComp
 $Comp
-L GND #PWR14
+L GND #PWR018
 U 1 1 5788F1B2
 P 5550 2150
-F 0 "#PWR14" H 5550 1900 50  0001 C CNN
+F 0 "#PWR018" H 5550 1900 50  0001 C CNN
 F 1 "GND" H 5555 1977 50  0000 C CNN
 F 2 "" H 5550 2150 50  0000 C CNN
@@
 $EndComp
 $Comp
-L GND #PWR18
+L GND #PWR019
 U 1 1 5788FD51
 P 8950 2450
-F 0 "#PWR18" H 8950 2200 50  0001 C CNN
+F 0 "#PWR019" H 8950 2200 50  0001 C CNN
 F 1 "GND" H 8955 2277 50  0000 C CNN
 F 2 "" H 8950 2450 50  0000 C CNN
@@
 $EndComp
 $Comp
-L +5V #PWR17
+L +5V #PWR020
 U 1 1 5788FE88
 P 8950 1300
-F 0 "#PWR17" H 8950 1150 50  0001 C CNN
+F 0 "#PWR020" H 8950 1150 50  0001 C CNN
 F 1 "+5V" H 8965 1473 50  0000 C CNN
 F 2 "" H 8950 1300 50  0000 C CNN
@@
 $EndComp
 $Comp
-L +5V #PWR15
+L +5V #PWR021
 U 1 1 5788FEE9
 P 6050 1600
-F 0 "#PWR15" H 6050 1450 50  0001 C CNN
+F 0 "#PWR021" H 6050 1450 50  0001 C CNN
 F 1 "+5V" H 6065 1773 50  0000 C CNN
 F 2 "" H 6050 1600 50  0000 C CNN
@@
 $EndComp
 $Comp
-L +5V #PWR6
+L +5V #PWR022
 U 1 1 5789013C
 P 2550 5100
-F 0 "#PWR6" H 2550 4950 50  0001 C CNN
+F 0 "#PWR022" H 2550 4950 50  0001 C CNN
 F 1 "+5V" H 2565 5273 50  0000 C CNN
 F 2 "" H 2550 5100 50  0000 C CNN
@@
 Text Notes 4350 7700 0    157  ~ 31
 FT232, USB & Lights
-Connection ~ 3800 4350
-Wire Wire Line
-	4050 4350 3800 4350
-Wire Wire Line
-	4050 3900 4050 4350
-Wire Wire Line
-	4000 3900 4050 3900
+Connection ~ 3700 4350
+Wire Wire Line
+	3950 4350 3700 4350
+Wire Wire Line
+	3950 3900 3950 4350
+Wire Wire Line
+	3900 3900 3950 3900
 Wire Notes Line
 	7000 6450 7000 2950
@@
 	1600 5300 1600 5200
 Wire Wire Line
-	3800 4300 3800 4450
+	3700 4300 3700 4450
 Connection ~ 3400 4400
 Wire Wire Line
@@
 	2500 1550 2500 1850
 $Comp
-L PWR_FLAG #FLG3
+L PWR_FLAG #FLG023
 U 1 1 57891E0F
 P 8850 4950
-F 0 "#FLG3" H 8850 5045 50  0001 C CNN
+F 0 "#FLG023" H 8850 5045 50  0001 C CNN
 F 1 "PWR_FLAG" V 8850 5128 50  0000 L CNN
 F 2 "" H 8850 4950 50  0000 C CNN
@@
 	2100 5300 2900 5300
 Text Label 3500 4500 1    60   ~ 0
-Dm
+D-
 Text Label 3600 4500 1    60   ~ 0
-Dp
+D+
 NoConn ~ 2900 6100
 $Comp
@@
 Wire Wire Line
 	4900 4150 4900 4200
+$Comp
+L USB_A P1
+U 1 1 58FD21E5
+P 3600 4000
+F 0 "P1" H 3626 4416 50  0000 C CNN
+F 1 "USB_A" H 3626 4325 50  0000 C CNN
+F 2 "PadsLib:MC32603_USB_A" H 3626 4234 50  0000 C CNN
+F 3 "" V 3550 3900 50  0000 C CNN
+	1    3600 4000
+	1    0    0    -1
+$EndComp
+$Comp
+L PWR_FLAG #FLG024
+U 1 1 58FD2766
+P 3050 4350
+F 0 "#FLG024" H 3050 4445 50  0001 C CNN
+F 1 "PWR_FLAG" H 3050 4574 50  0000 C CNN
+F 2 "" H 3050 4350 50  0000 C CNN
+F 3 "" H 3050 4350 50  0000 C CNN
+	1    3050 4350
+	1    0    0    -1
+$EndComp
+Wire Wire Line
+	3050 4350 3050 4400
+Connection ~ 3050 4400
 $EndSCHEMATC

Commit message: Another stupid mistake corrected..
Connections:
- net +5V: no longer U2.2 (A)
- net GND: now also U2.2 (A)
Changed lines of the file:
@@
 Title "FelinæPurr"
 Date "2016-07-15"
-Rev "1.1"
+Rev "1.1A"
 Comp "986-Studio"
 Comment1 ""
@@
 Wire Wire Line
 	8750 2000 9550 2000
-Connection ~ 6150 1750
-Wire Wire Line
-	6150 1750 6150 2000
 Wire Wire Line
 	5550 2100 5550 2150
@@
 	3050 4350 3050 4400
 Connection ~ 3050 4400
+$Comp
+L GND #PWR?
+U 1 1 58FD2B50
+P 6150 2150
+F 0 "#PWR?" H 6150 1900 50  0001 C CNN
+F 1 "GND" H 6155 1977 50  0000 C CNN
+F 2 "" H 6150 2150 50  0000 C CNN
+F 3 "" H 6150 2150 50  0000 C CNN
+	1    6150 2150
+	1    0    0    -1
+$EndComp
+Wire Wire Line
+	6150 2150 6150 2000
 $EndSCHEMATC
