File: FelinaePurr.sch (KiCad schematic (older format))
At the start: 24 parts, among them P1 USB_A, P2 JACK, U1 FT232RL, U2 SN74LVC1G125-Q1

Commit message: Add 2.5 jack
Parts:
- added P3: JACK, PadsLib:JACK2.5, symbol CONN_01X03
- added P4, P5: MECANICAL, PadsLib:2mmHole, symbol CONN_01X01
- D1, D2, D3, D4: symbol LED -> LED-RESCUE-FelinaePurr
- P1: symbol USB_A -> USB_A-RESCUE-FelinaePurr
- P2: value JACK -> PCB
Connections:
- wire segments 79 -> 84
- no-connect marks 14 -> 16
Other:
- note added: "TIP\nBASE\nINNER"
- moved on the sheet: P2
Changed lines of the file:
@@
 EESchema Schematic File Version 2
+LIBS:FelinaePurr-rescue
 LIBS:power
 LIBS:device
@@
 L CONN_01X03 P2
 U 1 1 5788BF2B
-P 9400 4850
-F 0 "P2" H 9478 4891 50  0000 L CNN
-F 1 "JACK" H 9478 4800 50  0000 L CNN
-F 2 "Pin_Headers:Pin_Header_Straight_1x03" H 9400 4850 50  0001 C CNN
-F 3 "" H 9400 4850 50  0000 C CNN
-	1    9400 4850
+P 9400 4050
+F 0 "P2" H 9478 4091 50  0000 L CNN
+F 1 "PCB" H 9478 4000 50  0000 L CNN
+F 2 "Pin_Headers:Pin_Header_Straight_1x03" H 9400 4050 50  0001 C CNN
+F 3 "" H 9400 4050 50  0000 C CNN
+	1    9400 4050
 	1    0    0    -1
 $EndComp
@@
 L +5VL #PWR05
 U 1 1 5788C270
-P 9050 4650
-F 0 "#PWR05" H 9050 4500 50  0001 C CNN
-F 1 "+5VL" H 9065 4823 50  0000 C CNN
-F 2 "" H 9050 4650 50  0000 C CNN
-F 3 "" H 9050 4650 50  0000 C CNN
-	1    9050 4650
+P 9050 3850
+F 0 "#PWR05" H 9050 3700 50  0001 C CNN
+F 1 "+5VL" H 9065 4023 50  0000 C CNN
+F 2 "" H 9050 3850 50  0000 C CNN
+F 3 "" H 9050 3850 50  0000 C CNN
+	1    9050 3850
 	1    0    0    -1
 $EndComp
@@
 L GND #PWR06
 U 1 1 5788C2A8
-P 9050 5050
-F 0 "#PWR06" H 9050 4800 50  0001 C CNN
-F 1 "GND" H 9055 4877 50  0000 C CNN
-F 2 "" H 9050 5050 50  0000 C CNN
-F 3 "" H 9050 5050 50  0000 C CNN
-	1    9050 5050
-	1    0    0    -1
-$EndComp
-Text Label 8850 4850 0    60   ~ 0
+P 9050 4250
+F 0 "#PWR06" H 9050 4000 50  0001 C CNN
+F 1 "GND" H 9055 4077 50  0000 C CNN
+F 2 "" H 9050 4250 50  0000 C CNN
+F 3 "" H 9050 4250 50  0000 C CNN
+	1    9050 4250
+	1    0    0    -1
+$EndComp
+Text Label 8850 4050 0    60   ~ 0
 RXTXout
-Text Notes 9650 5000 0    60   ~ 0
+Text Notes 9650 4200 0    60   ~ 0
 TIP\nINNER\nBASE
 $Comp
 L PWR_FLAG #FLG07
 U 1 1 5788C38F
-P 8850 4750
-F 0 "#FLG07" H 8850 4845 50  0001 C CNN
-F 1 "PWR_FLAG" V 8850 4928 50  0000 L CNN
-F 2 "" H 8850 4750 50  0000 C CNN
-F 3 "" H 8850 4750 50  0000 C CNN
-	1    8850 4750
+P 8850 3950
+F 0 "#FLG07" H 8850 4045 50  0001 C CNN
+F 1 "PWR_FLAG" V 8850 4128 50  0000 L CNN
+F 2 "" H 8850 3950 50  0000 C CNN
+F 3 "" H 8850 3950 50  0000 C CNN
+	1    8850 3950
 	0    -1   -1   0
 $EndComp
@@
 NoConn ~ 4100 5650
 $Comp
-L LED D1
+L LED-RESCUE-FelinaePurr D1
 U 1 1 5788D434
 P 4300 4800
@@
 $EndComp
 $Comp
-L LED D2
+L LED-RESCUE-FelinaePurr D2
 U 1 1 5788D49B
 P 4600 4800
@@
 $EndComp
 $Comp
-L LED D3
+L LED-RESCUE-FelinaePurr D3
 U 1 1 5788DACE
 P 4900 4800
@@
 $EndComp
 $Comp
-L LED D4
+L LED-RESCUE-FelinaePurr D4
 U 1 1 5788DBDE
 P 5200 4800
@@
 Wire Wire Line
 	5550 1750 6250 1750
-Connection ~ 9050 4750
-Wire Wire Line
-	9050 4950 9050 5050
-Wire Wire Line
-	8850 4950 9200 4950
-Wire Wire Line
-	8850 4850 9200 4850
-Wire Wire Line
-	9050 4750 9050 4650
-Wire Wire Line
-	8850 4750 9200 4750
+Connection ~ 9050 3950
+Wire Wire Line
+	9050 4150 9050 4250
+Wire Wire Line
+	8850 4150 9200 4150
+Wire Wire Line
+	8850 4050 9200 4050
+Wire Wire Line
+	9050 3950 9050 3850
+Wire Wire Line
+	8850 3950 9200 3950
 Connection ~ 2500 1750
 Wire Wire Line
@@
 L PWR_FLAG #FLG023
 U 1 1 57891E0F
-P 8850 4950
-F 0 "#FLG023" H 8850 5045 50  0001 C CNN
-F 1 "PWR_FLAG" V 8850 5128 50  0000 L CNN
-F 2 "" H 8850 4950 50  0000 C CNN
-F 3 "" H 8850 4950 50  0000 C CNN
-	1    8850 4950
+P 8850 4150
+F 0 "#FLG023" H 8850 4245 50  0001 C CNN
+F 1 "PWR_FLAG" V 8850 4328 50  0000 L CNN
+F 2 "" H 8850 4150 50  0000 C CNN
+F 3 "" H 8850 4150 50  0000 C CNN
+	1    8850 4150
 	0    -1   -1   0
 $EndComp
-Connection ~ 9050 4950
+Connection ~ 9050 4150
 $Comp
 L C C6
@@
 	4900 4150 4900 4200
 $Comp
-L USB_A P1
+L USB_A-RESCUE-FelinaePurr P1
 U 1 1 58FD21E5
 P 3600 4000
@@
 Connection ~ 3050 4400
 $Comp
-L GND #PWR?
+L GND #PWR025
 U 1 1 58FD2B50
 P 6150 2150
-F 0 "#PWR?" H 6150 1900 50  0001 C CNN
+F 0 "#PWR025" H 6150 1900 50  0001 C CNN
 F 1 "GND" H 6155 1977 50  0000 C CNN
 F 2 "" H 6150 2150 50  0000 C CNN
@@
 Wire Wire Line
 	6150 2150 6150 2000
+$Comp
+L CONN_01X03 P3
+U 1 1 59889BD9
+P 9400 5100
+F 0 "P3" H 9400 5300 50  0000 C CNN
+F 1 "JACK" V 9500 5100 50  0000 C CNN
+F 2 "PadsLib:JACK2.5" H 9400 5100 50  0001 C CNN
+F 3 "" H 9400 5100 50  0000 C CNN
+	1    9400 5100
+	1    0    0    -1
+$EndComp
+Text Notes 9550 5250 0    60   ~ 0
+TIP\nBASE\nINNER
+Wire Wire Line
+	9200 5000 9050 5000
+Wire Wire Line
+	9050 5000 9050 4900
+Wire Wire Line
+	8850 5200 9200 5200
+Text Label 8850 5200 0    60   ~ 0
+RXTXout
+Wire Wire Line
+	9200 5100 8750 5100
+Wire Wire Line
+	8750 5100 8750 5250
+$Comp
+L GND #PWR026
+U 1 1 5988A104
+P 8750 5250
+F 0 "#PWR026" H 8750 5000 50  0001 C CNN
+F 1 "GND" H 8750 5100 50  0000 C CNN
+F 2 "" H 8750 5250 50  0000 C CNN
+F 3 "" H 8750 5250 50  0000 C CNN
+	1    8750 5250
+	1    0    0    -1
+$EndComp
+$Comp
+L +5VL #PWR027
+U 1 1 5988A1F9
+P 9050 4900
+F 0 "#PWR027" H 9050 4750 50  0001 C CNN
+F 1 "+5VL" H 9050 5040 50  0000 C CNN
+F 2 "" H 9050 4900 50  0000 C CNN
+F 3 "" H 9050 4900 50  0000 C CNN
+	1    9050 4900
+	1    0    0    -1
+$EndComp
+$Comp
+L CONN_01X01 P4
+U 1 1 5988A54D
+P 7450 6350
+F 0 "P4" H 7450 6450 50  0000 C CNN
+F 1 "MECANICAL" V 7550 6350 50  0000 C CNN
+F 2 "PadsLib:2mmHole" H 7450 6350 50  0001 C CNN
+F 3 "" H 7450 6350 50  0000 C CNN
+	1    7450 6350
+	0    1    1    0
+$EndComp
+$Comp
+L CONN_01X01 P5
+U 1 1 5988A5A8
+P 7950 6350
+F 0 "P5" H 7950 6450 50  0000 C CNN
+F 1 "MECANICAL" V 8050 6350 50  0000 C CNN
+F 2 "PadsLib:2mmHole" H 7950 6350 50  0001 C CNN
+F 3 "" H 7950 6350 50  0000 C CNN
+	1    7950 6350
+	0    1    1    0
+$EndComp
+NoConn ~ 7950 6150
+NoConn ~ 7450 6150
+Wire Notes Line
+	7000 5800 8550 5800
+Wire Notes Line
+	8550 5800 8550 6450
 $EndSCHEMATC
